File: ECAD/color-sensor-2026/color-sensor-2026.kicad_pcb (KiCad board)
At the start: 2 copper layers, 10 parts, among them SW2 Sensor, U1 ATtiny412-SS

Commit message: V1 color sensor
Parts:
- removed C2: C_Small, Capacitor_SMD:C_1206_3216Metric_Pad1.33x1.80mm_HandSolder
- removed SW2: Sensor, Button_Switch_THT:SW_XKB_DM1-16UP-1
- added H1: MountingHole_Pad, MountingHole:MountingHole_3.2mm_M3_Pad_Via, F.Cu at (70.0, 88.0)
- added J1: Conn_01x05, Connector_PinHeader_2.54mm:PinHeader_1x05_P2.54mm_Horizontal, F.Cu at (78.1, 108.0)
- moved C1 99.4 mm to (68.3, 102.2), turned to 90 degrees
- moved U1 95.4 mm to (72.3, 102.1), turned to 90 degrees
- moved JP2 87.6 mm to (76.6, 102.1), turned to -90 degrees
- moved R1 82.4 mm to (75.1, 88.0)
- moved D1 78.1 mm to (73.0, 94.5), turned to 180 degrees
- moved R3 75.9 mm to (68.2, 94.8), turned to 90 degrees
- moved R2 67.3 mm to (78.4, 102.1), turned to -90 degrees
- moved R4 66.2 mm to (77.9, 94.8), turned to 90 degrees
Connections:
- U1 pad 5: Net-(U1-PA2) -> unconnected-(U1-PA2-Pad5)
Routing:
- net +3.3V: track 0.00 -> 38.1 mm
- net Net-(U1-PA1): track 0.00 -> 25.4 mm, vias 0 -> 1
- net Net-(JP2-A): track 0.00 -> 7.35 mm
- net /UPDI: track 0.00 -> 6.71 mm
- net Net-(U1-PA3): track 0.00 -> 5.95 mm
- net GND: track 0.00 -> 5.49 mm, vias 0 -> 11
- net /RX: track 0.00 -> 4.84 mm
- net Net-(D1-DIN): track 0.00 -> 4.51 mm
- net /TX/DAC: track 0.00 -> 3.95 mm
- added copper zone on B.Cu, net GND
- added copper zone on F.Cu, net GND
Other:
- board outline added: 14 x 35 mm
