File: ECAD/color-sensor-2026/color-sensor-2026.kicad_sch (KiCad schematic)
At the start: 10 parts, among them SW2 Sensor, U1 ATtiny412-SS

Commit message: V1 color sensor
Parts:
- removed C2: C_Small, Capacitor_SMD:C_1206_3216Metric_Pad1.33x1.80mm_HandSolder, symbol Device:C_Small
- removed SW2: Sensor, Button_Switch_THT:SW_XKB_DM1-16UP-1, symbol Switch:SW_Push
- added H1: MountingHole_Pad, MountingHole:MountingHole_3.2mm_M3_Pad_Via, symbol Mechanical:MountingHole_Pad
- added J1: Conn_01x05, Connector_PinHeader_2.54mm:PinHeader_1x05_P2.54mm_Horizontal, symbol Connector_Generic:Conn_01x05
Connections:
- net +3.3V: now also J1.4 (Pin_4)
- net GND: now also H1.1, J1.5 (Pin_5)
- net RX: now also J1.2 (Pin_2)
- net TX/DAC: now also J1.3 (Pin_3)
- net UPDI: now also J1.1 (Pin_1)
- no-connect marks 1 -> 2
Other:
- moved on the sheet: R1, R4

Commit message: firmware - serial version
Parts:
- R1: value LDR07 -> LDR07 - GL5516
Changed lines of the file:
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@@
 			)
 		)
-		(property "Value" "LDR07"
+		(property "Value" "LDR07 - GL5516"
 			(at 139.192 51.562 0)
 			(effects
