File: ECAD/I2C-GPIO-extenseur/I2C-GPIO-extenseur.kicad_pcb (KiCad board)
At the start: 2 copper layers, 58 x 38 mm, 97 parts, among them J1 Conn_01x03, J10 Conn_01x03, J11 Conn_01x03, J12 Conn_01x03, J13 Conn_01x03, J14 Conn_01x03, J15 Conn_01x03, J16 Conn_01x03, J17 Conn_01x03, J18 Conn_01x04, J19 Conn_01x04, J2 Conn_01x02, J3 Conn_01x03, J4 Conn_01x03, J5 Conn_01x03, J6 Conn_01x03, J7 Conn_01x03, J8 Conn_01x03, J9 Conn_01x03, U1 PCA9685PW

Commit message: update size and position
Parts:
- removed C1: C_Polarized_Small, Capacitor_THT:CP_Radial_D10.0mm_P5.00mm
- removed C4: 10uF, Capacitor_SMD:C_1206_3216Metric_Pad1.33x1.80mm_HandSolder
- removed J10, J11, J12, J13, J14, J15, J16, J17: Conn_01x03, Connector_PinHeader_2.54mm:PinHeader_1x03_P2.54mm_Vertical
- removed JP5, JP6: SolderJumper_2_Open, Jumper:SolderJumper-2_P1.3mm_Open_RoundedPad1.0x1.5mm
- removed R11, R12, R13, R14, R15, R16, R17, R3, R4, R5, R6, R7, R8, R9: 220, Resistor_SMD:R_1206_3216Metric_Pad1.30x1.75mm_HandSolder
- removed R20, R25, R26, R27: 10k, Resistor_SMD:R_1206_3216Metric_Pad1.30x1.75mm_HandSolder
- removed U1: PCA9685PW, Package_SO:TSSOP-28_4.4x9.7mm_P0.65mm
- added C2: 10uF, Capacitor_SMD:C_1206_3216Metric_Pad1.33x1.80mm_HandSolder, F.Cu at (88.1, 75.8)
- added U2: ATtiny3216-S, Package_SO:SOIC-20W_7.5x12.8mm_P1.27mm, F.Cu at (87.8, 83.7)
- J2: value Conn_01x02 -> Conn_01x05; footprint Connector_Molex:Molex_KK-396_A-41791-0002_1x02_P3.96mm_Vertical -> Connector_PinHeader_2.54mm:PinHeader_1x05_P2.54mm_Vertical
- R1: value 1k -> 10k
- R10: value 220 -> 1k; moved to B.Cu
- R2: value 220 -> 4k7
- moved J2 41.0 mm to (103.0, 76.0), turned to 0 degrees
- moved R2 37.5 mm to (98.7, 83.1), turned to 0 degrees
- moved G*** 37.0 mm to (129.0, 85.2)
- moved J1 33.8 mm to (65.9, 73.0), turned to -90 degrees
- moved R1 32.1 mm to (95.7, 81.5), turned to 0 degrees
- moved D1 32.0 mm to (97.8, 78.5), turned to 180 degrees
- moved R22 30.0 mm to (95.7, 89.2), turned to 0 degrees
- moved R23 27.2 mm to (95.7, 86.6), turned to 0 degrees
- moved JP1 26.9 mm to (91.5, 89.2), turned to 180 degrees
- moved J5 26.3 mm to (65.9, 70.5), turned to -90 degrees
- moved R24 24.5 mm to (95.7, 84.1), turned to 0 degrees
- moved J7 24.3 mm to (65.9, 85.7), turned to -90 degrees
- moved JP2 23.7 mm to (91.5, 86.6), turned to 180 degrees
- moved JP3 20.7 mm to (91.5, 84.1), turned to 180 degrees
- moved J4 20.7 mm to (65.9, 79.4), turned to -90 degrees
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Connections:
- J1 pad 1: Net-(J1-Pin_1) -> GPIO_1
- J1 pad 2: +5VP -> +3.3V
- J2 pad 1: +5VP -> GND
- J2 pad 2: GND -> RX
- J3 pad 1: Net-(J3-Pin_1) -> GPIO_2
- J3 pad 2: +5VP -> +3.3V
- J4 pad 1: Net-(J4-Pin_1) -> GPIO_3
- J4 pad 2: +5VP -> +3.3V
- J5 pad 1: Net-(J5-Pin_1) -> GPIO_0
- J5 pad 2: +5VP -> +3.3V
- J6 pad 1: Net-(J6-Pin_1) -> GPIO_4
- J6 pad 2: +5VP -> +3.3V
- J7 pad 1: Net-(J7-Pin_1) -> GPIO_5
- J7 pad 2: +5VP -> +3.3V
- J8 pad 1: Net-(J8-Pin_1) -> GPIO_6
- J8 pad 2: +5VP -> +3.3V
- J9 pad 1: Net-(J9-Pin_1) -> GPIO_7
- J9 pad 2: +5VP -> +3.3V
- R1 pad 1: +5VP -> A3
- R1 pad 2: Net-(D1-A) -> GND
- R10 pad 1: Net-(J7-Pin_1) -> Net-(U2-PA3)
- R10 pad 2: Act_08 -> Net-(D1-A)
- R2 pad 1: Net-(J5-Pin_1) -> Net-(U2-~{RESET}/PA0)
- R2 pad 2: Act_00 -> UPDI
Routing:
- net +5VP: track 97.6 -> 0.00 mm
- net +3.3V: track 75.0 -> 0.00 mm
- net SDA: track 35.7 -> 0.00 mm
- net SCL: track 28.8 -> 0.00 mm
- net Act_00: track 26.2 -> 0.00 mm
- net Act_01: track 23.4 -> 0.00 mm
- net A0: track 21.0 -> 0.00 mm, vias 1 -> 0
- net Act_02: track 20.6 -> 0.00 mm
- net A1: track 18.2 -> 0.00 mm, vias 1 -> 0
- net Act_03: track 17.8 -> 0.00 mm
- net A2: track 15.4 -> 0.00 mm, vias 1 -> 0
- net A5: track 12.9 -> 0.00 mm, vias 1 -> 0
- net A3: track 12.5 -> 0.00 mm, vias 1 -> 0
- net Act_04: track 12.0 -> 0.00 mm
- net Net-(U1-~{OE}): track 11.5 -> 0.00 mm
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Other:
- board size 58 x 38 mm -> 58 x 30 mm
