File: ECAD/I2C-GPIO-expander-PCF/I2C-GPIO-expander-PCF.kicad_pcb (KiCad board)
At the start: 2 copper layers, 58 x 25 mm, 62 parts, among them J1 Conn_01x03, J18 Conn_01x04, J19 Conn_01x04, J3 Conn_01x03, J4 Conn_01x03, J5 Conn_01x03, J6 Conn_01x03, J7 Conn_01x03, J8 Conn_01x03, J9 Conn_01x03, U1 PCF8574AT

Commit message: Silkscreen
Parts:
- removed the G*** at (49.0, 73.0)
- removed the G*** at (49.0, 97.0)
- removed the G*** at (52.4, 86.4)
- removed the G*** at (105.0, 97.0)
- removed the G*** at (58.3, 77.7)
- removed the G*** at (129.7, 63.4)
- removed the G*** at (58.3, 75.0)
- removed the G*** at (105.0, 73.0)
- removed kibuzzard-67954B90: G***, kibuzzard-67954B90
- removed kibuzzard-67954C44: G***, kibuzzard-67954C44
- removed kibuzzard-67954C4A: G***, kibuzzard-67954C4A
- removed kibuzzard-67954C57: G***, kibuzzard-67954C57
- removed kibuzzard-67954C5E: G***, kibuzzard-67954C5E
- removed kibuzzard-67954C66: G***, kibuzzard-67954C66
- removed kibuzzard-67954E34: G***, kibuzzard-67954E34
- removed kibuzzard-67954E39: G***, kibuzzard-67954E39
- removed kibuzzard-67954E3F: G***, kibuzzard-67954E3F
- removed the kibuzzard-67954E7A at (73.7, 72.6)
- removed the kibuzzard-67954E99 at (87.6, 72.4)
- removed the kibuzzard-67954EA0 at (90.2, 72.4)
- added kibuzzard-67954D1A: G***, kibuzzard-67954D1A, F.Cu at (87.7, 74.8)
- added kibuzzard-67954D30: G***, kibuzzard-67954D30, F.Cu at (90.3, 74.8)
- added kibuzzard-698C5220: G***, kibuzzard-698C5220, F.Cu at (62.6, 78.5)
- added kibuzzard-698C52C9: G***, kibuzzard-698C52C9, F.Cu at (67.5, 68.0)
- added kibuzzard-698C52CF: G***, kibuzzard-698C52CF, F.Cu at (67.6, 70.5)
- added kibuzzard-698C52D4: G***, kibuzzard-698C52D4, F.Cu at (67.6, 74.0)
- added kibuzzard-698C52DA: G***, kibuzzard-698C52DA, F.Cu at (67.6, 76.6)
- added kibuzzard-698C52E2: G***, kibuzzard-698C52E2, F.Cu at (67.6, 80.5)
- added kibuzzard-698C52E7: G***, kibuzzard-698C52E7, F.Cu at (67.6, 83.0)
- added kibuzzard-698C52ED: G***, kibuzzard-698C52ED, F.Cu at (67.6, 86.4)
- added kibuzzard-698C52F2: G***, kibuzzard-698C52F2, F.Cu at (67.6, 88.9)
- added kibuzzard-698C538A: G***, kibuzzard-698C538A, F.Cu at (87.5, 81.9)
- moved G*** 76.2 mm to (53.2, 77.0)
- moved G*** 25.2 mm to (102.5, 80.1)
- moved G*** 25.1 mm to (58.0, 76.6)
- moved kibuzzard-67954E00 19.6 mm to (83.7, 86.6)
- moved kibuzzard-67954E2A 15.2 mm to (81.2, 86.6)
- moved kibuzzard-67954E2F 11.3 mm to (78.6, 86.6)
Other:
- board text added: "Karibous 2025-26"
- board text added: "Open = 0 Close = 1 Base = 0x20"
- board text removed: "+"
- board text removed: "Carte Servo"
- board text removed: "Karibous 2024-25"
- board text removed: "Open = 0 Close = 1 Base = 0x40"
